File: HSC_Alice/HSC_Alice.kicad_pcb (KiCad board)
At the start: 2 copper layers, 481.7 x 142.6 mm, 211 parts, among them U2 Elite-C

Commit message: Bug Fixes
Fixed wiring 90Deg angles

Reworked Gerber Files
Parts:
- moved MX91 2.00 mm to (-256.1, 64.3)
- moved D101 2.00 mm to (-229.5, 126.2)
- moved D102 2.00 mm to (-205.7, 145.3)
- moved D103 2.00 mm to (-205.7, 64.3)
- moved D104 2.00 mm to (-224.8, 88.1)
- moved D105 2.00 mm to (-215.2, 107.2)
- moved D84 2.00 mm to (-258.1, 164.4)
- moved D87 2.00 mm to (-272.4, 107.2)
- moved D88 2.00 mm to (-267.6, 126.2)
- moved D89 2.00 mm to (-267.6, 145.3)
- moved D90 2.00 mm to (-234.3, 164.4)
- moved D91 2.00 mm to (-265.6, 64.3)
- moved D92 2.00 mm to (-262.9, 88.2)
- moved D93 2.00 mm to (-253.4, 107.2)
- moved D94 2.00 mm to (-248.6, 126.2)
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Routing:
- net Net-(D89-Pad2): track 0.00 -> 14.2 mm
- net Net-(D36-Pad2): track 0.00 -> 10.6 mm
- net Row4: track 567.3 -> 557.8 mm, vias 7 -> 6
- net Row3: track 521.5 -> 519.0 mm
- net Col3: track 214.7 -> 212.4 mm
- net Col7: track 229.4 -> 231.3 mm
- net Col8: track 273.2 -> 275.1 mm
- net Col12: track 347.2 -> 349.0 mm
- net Net-(U2-Pad4): track 0.00 -> 1.78 mm
- net Net-(U2-Pad3): track 0.00 -> 1.78 mm
- net Net-(U2-Pad23): track 0.00 -> 1.78 mm
- net Net-(U2-Pad22): track 0.00 -> 1.78 mm
- net Net-(U2-Pad21): track 0.00 -> 1.78 mm
- net Col4: track 204.9 -> 206.7 mm
- net Col11: track 340.9 -> 342.7 mm
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Other:
- board size 481.7 x 142.6 mm -> 479.3 x 144.1 mm

Commit message: Update HSC_Alice.kicad_pcb
Fixed routing errors
Routing:
- net Row1: track 535.0 -> 529.6 mm
- net Col16: track 442.3 -> 438.9 mm
- net Row5: track 639.4 -> 637.4 mm
Changed lines of the file:
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@@
     (thickness 1.6)
     (drawings 14)
-    (tracks 1042)
+    (tracks 1044)
     (zones 0)
     (modules 211)
@@
   (segment (start -653.963 83.638) (end -649.788 83.638) (width 0.254) (layer F.Cu) (net 3))
   (via (at -565.9755 89.788) (size 0.8) (drill 0.4) (layers F.Cu B.Cu) (net 4))
-  (via (at -608.7872 92.1004) (size 0.8) (drill 0.4) (layers F.Cu B.Cu) (net 4))
-  (segment (start -644.6256 92.1004) (end -608.7872 92.1004) (width 0.254) (layer B.Cu) (net 4))
-  (segment (start -646.938 89.788) (end -644.6256 92.1004) (width 0.254) (layer B.Cu) (net 4))
   (via (at -608.838 108.838) (size 0.8) (drill 0.4) (layers F.Cu B.Cu) (net 4))
-  (segment (start -608.7872 108.7872) (end -608.838 108.838) (width 0.254) (layer F.Cu) (net 4))
-  (segment (start -608.7872 92.1004) (end -608.7872 108.7872) (width 0.254) (layer F.Cu) (net 4))
   (via (at -574.167 115.0874) (size 0.8) (drill 0.4) (layers F.Cu B.Cu) (net 4))
   (segment (start -279.9334 89.8134) (end -279.262499 90.484301) (width 0.254) (layer B.Cu) (net 4))
@@
   (via (at -557.5808 98.806) (size 0.8) (drill 0.4) (layers F.Cu B.Cu) (net 7))
   (via (at -626.6688 98.5774) (size 0.8) (drill 0.4) (layers F.Cu B.Cu) (net 7))
-  (segment (start -626.4402 98.806) (end -626.6688 98.5774) (width 0.254) (layer B.Cu) (net 7))
-  (segment (start -557.5808 98.806) (end -626.4402 98.806) (width 0.254) (layer B.Cu) (net 7))
   (via (at -627.888 108.838) (size 0.8) (drill 0.4) (layers F.Cu B.Cu) (net 7))
   (segment (start -627.888 99.7966) (end -627.888 108.838) (width 0.254) (layer F.Cu) (net 7))
@@
   (segment (start -357.442784 183.538035) (end -320.399228 183.538035) (width 0.254) (layer B.Cu) (net 12))
   (segment (start -363.252968 189.348219) (end -357.442784 183.538035) (width 0.254) (layer B.Cu) (net 12))
-  (segment (start -293.105368 166.0134) (end -258.05105 166.0134) (width 0.254) (layer B.Cu) (net 12))
   (segment (start -300.881305 175.789337) (end -291.105368 166.0134) (width 0.254) (layer B.Cu) (net 12))
   (segment (start -312.65053 175.789337) (end -300.881305 175.789337) (width 0.254) (layer B.Cu) (net 12))
@@
   (segment (start -601.627436 122.995001) (end -594.420001 122.995001) (width 0.254) (layer F.Cu) (net 4))
   (segment (start -608.838 108.838) (end -608.838 115.784437) (width 0.254) (layer F.Cu) (net 4))
+  (segment (start -644.6256 92.1004) (end -646.938 89.788) (width 0.254) (layer B.Cu) (net 4))
+  (segment (start -618.9726 92.1512) (end -644.6256 92.1004) (width 0.254) (layer B.Cu) (net 4))
+  (via (at -618.9726 92.1512) (size 0.8) (drill 0.4) (layers F.Cu B.Cu) (net 4))
+  (segment (start -608.7872 108.7872) (end -608.838 108.838) (width 0.254) (layer F.Cu) (net 4))
+  (segment (start -611.8098 105.2322) (end -608.7872 108.7872) (width 0.254) (layer F.Cu) (net 4))
+  (segment (start -611.7844 97.2058) (end -611.8098 105.2322) (width 0.254) (layer F.Cu) (net 4))
+  (segment (start -618.9726 92.1512) (end -611.7844 97.2058) (width 0.254) (layer F.Cu) (net 4))
   (segment (start -275.192723 113.622323) (end -272.3642 108.8136) (width 0.254) (layer B.Cu) (net 7))
   (segment (start -301.503134 113.622323) (end -275.192723 113.622323) (width 0.254) (layer B.Cu) (net 7))
@@
   (segment (start -557.5554 86.5378) (end -557.5554 98.7806) (width 0.254) (layer F.Cu) (net 7))
   (segment (start -557.5554 86.5378) (end -555.5488 86.5378) (width 0.254) (layer F.Cu) (net 7))
+  (segment (start -625.2718 98.5774) (end -626.6688 98.5774) (width 0.254) (layer B.Cu) (net 7))
+  (segment (start -557.5808 98.806) (end -625.2718 98.5774) (width 0.254) (layer B.Cu) (net 7))
   (segment (start -298.048734 132.418323) (end -272.161 132.418323) (width 0.254) (layer B.Cu) (net 8))
   (segment (start -566.1914 165.7721) (end -565.9755 165.988) (width 0.254) (layer F.Cu) (net 8))
@@
   (segment (start -658.113 154.813) (end -657.185999 153.885999) (width 0.254) (layer B.Cu) (net 12))
   (segment (start -548.1574 117.3988) (end -548.1574 86.5378) (width 0.254) (layer F.Cu) (net 12))
+  (segment (start -291.1094 166.0144) (end -258.05105 166.0134) (width 0.254) (layer B.Cu) (net 12))
   (segment (start -590.678 114.173) (end -589.788 115.063) (width 0.254) (layer B.Cu) (net 20))
   (segment (start -604.393 114.173) (end -590.678 114.173) (width 0.254) (layer B.Cu) (net 20))
@@
   (segment (start -536.8804 71.2978) (end -532.6634 67.0808) (width 0.254) (layer F.Cu) (net 126))
   (segment (start -540.5374 71.2978) (end -536.8804 71.2978) (width 0.254) (layer F.Cu) (net 126))
-  (via (at -211.6262 142.9004) (size 0.8) (drill 0.4) (layers F.Cu B.Cu) (net 127))
-  (segment (start -211.4738 142.748) (end -211.6262 142.9004) (width 0.254) (layer B.Cu) (net 127))
-  (segment (start -199.993 142.748) (end -211.4738 142.748) (width 0.254) (layer B.Cu) (net 127))
-  (segment (start -211.6262 123.9832) (end -211.9114 123.698) (width 0.254) (layer F.Cu) (net 127))
-  (segment (start -211.6262 142.9004) (end -211.6262 123.9832) (width 0.254) (layer F.Cu) (net 127))
   (segment (start -228.5934 106.838334) (end -211.9114 123.520334) (width 0.254) (layer F.Cu) (net 127))
   (segment (start -211.9114 123.520334) (end -211.9114 123.698) (width 0.254) (layer F.Cu) (net 127))
@@
   (segment (start -536.8804 68.7578) (end -534.2382 66.1156) (width 0.254) (layer F.Cu) (net 127))
   (segment (start -540.5374 68.7578) (end -536.8804 68.7578) (width 0.254) (layer F.Cu) (net 127))
+  (segment (start -211.6262 123.9832) (end -211.9114 123.698) (width 0.254) (layer F.Cu) (net 127))
+  (segment (start -211.6262 136.6454) (end -211.6262 123.9832) (width 0.254) (layer F.Cu) (net 127))
+  (via (at -211.6262 136.6454) (size 0.8) (drill 0.4) (layers F.Cu B.Cu) (net 127))
+  (segment (start -204.6732 136.6266) (end -198.683 141.288) (width 0.254) (layer B.Cu) (net 127))
+  (segment (start -211.6262 136.6454) (end -204.6732 136.6266) (width 0.254) (layer B.Cu) (net 127))
   (segment (start -538.7594 58.5978) (end -535.9654 55.8038) (width 0.254) (layer F.Cu) (net 128))
   (segment (start -208.2334 69.516938) (end -208.2334 84.138) (width 0.254) (layer F.Cu) (net 128))
