File: HSC_Alice/HSC_Alice.kicad_pcb (KiCad board)
At the start: 2 copper layers, 76.2 x 38.1 mm, 24 parts, among them SW1 SW_Push, U1 ATmega32U4-AU, Y1 16MHz

Commit message: Numpad
Added Numpad Row and Col
Parts:
- removed C1, C2, C5, C7: 0.1uF, Capacitor_SMD:C_0805_2012Metric_Pad1.18x1.45mm_HandSolder
- removed C3, C4: 22pF, Capacitor_SMD:C_0805_2012Metric_Pad1.18x1.45mm_HandSolder
- removed C6: 1uF, Capacitor_SMD:C_0805_2012Metric_Pad1.18x1.45mm_HandSolder
- removed F1: 500mA, Fuse:Fuse_1206_3216Metric_Pad1.42x1.75mm_HandSolder
- removed R1, R2: 22, Resistor_SMD:R_0805_2012Metric_Pad1.20x1.40mm_HandSolder
- removed R3, R4: 10k, Resistor_SMD:R_0805_2012Metric_Pad1.20x1.40mm_HandSolder
- removed SW1: SW_Push, random-keyboard-parts:SKQG-1155865
- removed U1: ATmega32U4-AU, Package_QFP:TQFP-44_10x10mm_P0.8mm
- removed USB1: Molex-0548190589, random-keyboard-parts:Molex-0548190589
- removed Y1: 16MHz, Crystal:Crystal_SMD_3225-4Pin_3.2x2.5mm_HandSoldering
- added D10: D_Small, Diode_SMD:D_SOD-123, F.Cu at (-627.9, 126.2)
- added D100: D_Small, Diode_SMD:D_SOD-123, F.Cu at (-346.2, 126.9)
- added D101: D_Small, Diode_SMD:D_SOD-123, F.Cu at (-389.8, 191.6)
- added D102: D_Small, Diode_SMD:D_SOD-123, F.Cu at (-389.8, 195.0)
- added D103: D_Small, Diode_SMD:D_SOD-123, F.Cu at (-384.1, 191.6)
- added D104: D_Small, Diode_SMD:D_SOD-123, F.Cu at (-384.1, 195.0)
- added D105: D_Small, Diode_SMD:D_SOD-123, F.Cu at (-389.8, 198.3)
- added D106: D_Small, Diode_SMD:D_SOD-123, F.Cu at (-366.8, 205.0)
- added D11: D_Small, Diode_SMD:D_SOD-123, F.Cu at (-627.9, 145.3)
- added D12: D_Small, Diode_SMD:D_SOD-123, F.Cu at (-236.9, 207.1)
- added D13: D_Small, Diode_SMD:D_SOD-123, F.Cu at (-589.8, 88.1)
- added D14: D_Small, Diode_SMD:D_SOD-123, F.Cu at (-589.8, 116.7)
- added D15: D_Small, Diode_SMD:D_SOD-123, F.Cu at (-608.8, 126.2)
- added D16: D_Small, Diode_SMD:D_SOD-123, F.Cu at (-71.2, 38.0)
- added D17: D_Small, Diode_SMD:D_SOD-123, F.Cu at (-608.8, 154.8)
- added D18: D_Small, Diode_SMD:D_SOD-123, F.Cu at (-71.2, 34.7)
- added D19: D_Small, Diode_SMD:D_SOD-123, F.Cu at (-65.5, 28.0)
- added D20: D_Small, Diode_SMD:D_SOD-123, F.Cu at (-65.5, 24.6)
- added D21: D_Small, Diode_SMD:D_SOD-123, F.Cu at (-71.2, 31.3)
- added D22: D_Small, Diode_SMD:D_SOD-123, F.Cu at (-71.2, 28.0)
- added D23: D_Small, Diode_SMD:D_SOD-123, F.Cu at (-248.4, 207.1)
- added D24: D_Small, Diode_SMD:D_SOD-123, F.Cu at (-71.2, 24.6)
- added D25: D_Small, Diode_SMD:D_SOD-123, F.Cu at (-315.1, 205.0)
- added D26: D_Small, Diode_SMD:D_SOD-123, F.Cu at (-71.2, 41.4)
- added D27: D_Small, Diode_SMD:D_SOD-123, F.Cu at (-326.6, 191.6)
- added D28: D_Small, Diode_SMD:D_SOD-123, F.Cu at (-320.8, 205.0)
- added D29: D_Small, Diode_SMD:D_SOD-123, F.Cu at (-326.6, 205.0)
- added D30: D_Small, Diode_SMD:D_SOD-123, F.Cu at (-320.8, 201.7)
- added D31: D_Small, Diode_SMD:D_SOD-123, F.Cu at (-320.8, 198.3)
- added D32: D_Small, Diode_SMD:D_SOD-123, F.Cu at (-315.1, 195.0)
- added D33: D_Small, Diode_SMD:D_SOD-123, F.Cu at (-315.1, 191.6)
- added D34: D_Small, Diode_SMD:D_SOD-123, F.Cu at (-320.8, 195.0)
- added D35: D_Small, Diode_SMD:D_SOD-123, F.Cu at (-326.6, 201.7)
- added D36: D_Small, Diode_SMD:D_SOD-123, F.Cu at (-332.3, 205.0)
- added D37: D_Small, Diode_SMD:D_SOD-123, F.Cu at (-320.8, 191.6)
- added D38: D_Small, Diode_SMD:D_SOD-123, F.Cu at (-326.6, 198.3)
- added D39: D_Small, Diode_SMD:D_SOD-123, F.Cu at (-343.8, 198.3)
- added D40: D_Small, Diode_SMD:D_SOD-123, F.Cu at (-326.6, 195.0)
- added D41: D_Small, Diode_SMD:D_SOD-123, F.Cu at (-315.1, 198.3)
- added D42: D_Small, Diode_SMD:D_SOD-123, F.Cu at (-332.3, 198.3)
- added D43: D_Small, Diode_SMD:D_SOD-123, F.Cu at (-338.1, 205.0)
- added D44: D_Small, Diode_SMD:D_SOD-123, F.Cu at (-338.1, 201.7)
- added D45: D_Small, Diode_SMD:D_SOD-123, F.Cu at (-332.3, 195.0)
- added D46: D_Small, Diode_SMD:D_SOD-123, F.Cu at (-343.8, 205.0)
- added D47: D_Small, Diode_SMD:D_SOD-123, F.Cu at (-349.6, 205.0)
- added D48: D_Small, Diode_SMD:D_SOD-123, F.Cu at (-343.8, 201.7)
- added D49: D_Small, Diode_SMD:D_SOD-123, F.Cu at (-338.1, 198.3)
- added D5: D_Small, Diode_SMD:D_SOD-123, F.Cu at (-646.9, 145.3)
- added D50: D_Small, Diode_SMD:D_SOD-123, F.Cu at (-338.1, 195.0)
- added D51: D_Small, Diode_SMD:D_SOD-123, F.Cu at (-332.3, 191.6)
- added D52: D_Small, Diode_SMD:D_SOD-123, F.Cu at (-338.1, 191.6)
- added D53: D_Small, Diode_SMD:D_SOD-123, F.Cu at (-332.3, 201.7)
- added D54: D_Small, Diode_SMD:D_SOD-123, F.Cu at (-65.5, 34.7)
- added D55: D_Small, Diode_SMD:D_SOD-123, F.Cu at (-343.8, 195.0)
- added D56: D_Small, Diode_SMD:D_SOD-123, F.Cu at (-343.8, 191.6)
- added D57: D_Small, Diode_SMD:D_SOD-123, F.Cu at (-318.7, 167.3)
- added D58: D_Small, Diode_SMD:D_SOD-123, F.Cu at (-355.3, 205.0)
- added D59: D_Small, Diode_SMD:D_SOD-123, F.Cu at (-349.6, 198.3)
- added D6: D_Small, Diode_SMD:D_SOD-123, F.Cu at (-656.5, 154.8)
- added D60: D_Small, Diode_SMD:D_SOD-123, F.Cu at (-349.6, 195.0)
- added D61: D_Small, Diode_SMD:D_SOD-123, F.Cu at (-355.3, 201.7)
- added D62: D_Small, Diode_SMD:D_SOD-123, F.Cu at (-324.5, 167.3)
- added D63: D_Small, Diode_SMD:D_SOD-123, F.Cu at (-355.3, 198.3)
- added D64: D_Small, Diode_SMD:D_SOD-123, F.Cu at (-361.1, 205.0)
- added D65: D_Small, Diode_SMD:D_SOD-123, F.Cu at (-349.6, 191.6)
- added D66: D_Small, Diode_SMD:D_SOD-123, F.Cu at (-372.6, 198.3)
- added D67: D_Small, Diode_SMD:D_SOD-123, F.Cu at (-349.6, 201.7)
- added D68: D_Small, Diode_SMD:D_SOD-123, F.Cu at (-361.1, 198.3)
- added D69: D_Small, Diode_SMD:D_SOD-123, F.Cu at (-355.3, 195.0)
- added D7: D_Small, Diode_SMD:D_SOD-123, F.Cu at (-608.8, 88.1)
- added D70: D_Small, Diode_SMD:D_SOD-123, F.Cu at (-355.3, 191.6)
- added D71: D_Small, Diode_SMD:D_SOD-123, F.Cu at (-361.1, 195.0)
- added D72: D_Small, Diode_SMD:D_SOD-123, F.Cu at (-366.8, 201.7)
- added D73: D_Small, Diode_SMD:D_SOD-123, F.Cu at (-372.6, 205.0)
- added D74: D_Small, Diode_SMD:D_SOD-123, F.Cu at (-361.1, 191.6)
- added D75: D_Small, Diode_SMD:D_SOD-123, F.Cu at (-366.8, 198.3)
- added D76: D_Small, Diode_SMD:D_SOD-123, F.Cu at (-372.6, 201.7)
- added D77: D_Small, Diode_SMD:D_SOD-123, F.Cu at (-366.8, 195.0)
- added D78: D_Small, Diode_SMD:D_SOD-123, F.Cu at (-366.8, 191.6)
- added D79: D_Small, Diode_SMD:D_SOD-123, F.Cu at (-378.3, 201.7)
- added D8: D_Small, Diode_SMD:D_SOD-123, F.Cu at (-608.8, 107.2)
- added D80: D_Small, Diode_SMD:D_SOD-123, F.Cu at (-316.1, 69.7)
- added D81: D_Small, Diode_SMD:D_SOD-123, F.Cu at (-372.6, 195.0)
- added D82: D_Small, Diode_SMD:D_SOD-123, F.Cu at (-372.6, 191.6)
- added D83: D_Small, Diode_SMD:D_SOD-123, F.Cu at (-378.3, 198.3)
- added D84: D_Small, Diode_SMD:D_SOD-123, F.Cu at (-384.1, 205.0)
- added D85: D_Small, Diode_SMD:D_SOD-123, F.Cu at (-389.8, 205.0)
- added D86: D_Small, Diode_SMD:D_SOD-123, F.Cu at (-384.1, 201.7)
- added D87: D_Small, Diode_SMD:D_SOD-123, F.Cu at (-384.1, 198.3)
- added D88: D_Small, Diode_SMD:D_SOD-123, F.Cu at (-378.3, 195.0)
- added D89: D_Small, Diode_SMD:D_SOD-123, F.Cu at (-378.3, 191.6)
- added D9: D_Small, Diode_SMD:D_SOD-123, F.Cu at (-627.9, 107.2)
- added D90: D_Small, Diode_SMD:D_SOD-123, F.Cu at (-334.1, 147.1)
- added D91: D_Small, Diode_SMD:D_SOD-123, F.Cu at (-339.9, 147.1)
- added D92: D_Small, Diode_SMD:D_SOD-123, F.Cu at (-389.8, 201.7)
- added D93: D_Small, Diode_SMD:D_SOD-123, F.Cu at (-316.1, 66.3)
- added D94: D_Small, Diode_SMD:D_SOD-123, F.Cu at (-378.3, 205.0)
- added D95: D_Small, Diode_SMD:D_SOD-123, F.Cu at (-316.1, 73.0)
- added D96: D_Small, Diode_SMD:D_SOD-123, F.Cu at (-316.1, 76.4)
- added D97: D_Small, Diode_SMD:D_SOD-123, F.Cu at (-316.1, 79.7)
- added D98: D_Small, Diode_SMD:D_SOD-123, F.Cu at (-316.1, 83.1)
- added D99: D_Small, Diode_SMD:D_SOD-123, F.Cu at (-351.9, 126.9)
- added MX10: P5, MX_Alps_Hybrid:MX-1U-NoLED, F.Cu at (-637.4, 126.2)
- added MX100: \, MX_Alps_Hybrid:MX-1U-NoLED, F.Cu at (-288.7, 94.3)
- added MX101: ENTER, MX_Alps_Hybrid:MX-2.25U-NoLED, F.Cu at (-370.7, 53.9)
- added MX102: RGUI, MX_Alps_Hybrid:MX-1U-NoLED, F.Cu at (-225.6, 33.1)
- added MX103: DEL, MX_Alps_Hybrid:MX-1U-NoLED, F.Cu at (-382.6, 179.9)
- added MX104: BACKSPACE, MX_Alps_Hybrid:MX-2U-NoLED, F.Cu at (-373.1, 74.7)
- added MX105: \, MX_Alps_Hybrid:MX-1U-NoLED, F.Cu at (-318.4, 115.1)
- added MX106: ENTER, MX_Alps_Hybrid:MX-1U-NoLED, F.Cu at (-272.1, 134.7)
- added MX11: P2, MX_Alps_Hybrid:MX-1U-NoLED, F.Cu at (-637.4, 145.3)
- added MX12: P00, MX_Alps_Hybrid:MX-1U-NoLED, F.Cu at (-637.4, 164.3)
- added MX13: P-, MX_Alps_Hybrid:MX-1U-NoLED, F.Cu at (-599.3, 88.1)
- added MX14: P+, MX_Alps_Hybrid:MX-2U-NoLED, F.Cu at (-599.3, 116.7)
- added MX15: P6, MX_Alps_Hybrid:MX-1U-NoLED, F.Cu at (-618.4, 126.2)
- added MX16: P3, MX_Alps_Hybrid:MX-1U-NoLED, F.Cu at (-618.4, 145.3)
- added MX17: P., MX_Alps_Hybrid:MX-1U-NoLED, F.Cu at (-618.4, 164.3)
- added MX18: PENT, MX_Alps_Hybrid:MX-2U-NoLED, F.Cu at (-599.3, 154.8)
- added MX19: Escape, MX_Alps_Hybrid:MX-1U-NoLED, F.Cu at (-200.8, 175.1)
- added MX20: No, MX_Alps_Hybrid:MX-1U-NoLED, F.Cu at (-573.8, 88.0)
- added MX21: Up, MX_Alps_Hybrid:MX-1U-NoLED, F.Cu at (-555.5, 145.2)
- added MX22: Left, MX_Alps_Hybrid:MX-1U-NoLED, F.Cu at (-574.5, 164.2)
- added MX23: Down, MX_Alps_Hybrid:MX-1U-NoLED, F.Cu at (-555.5, 164.2)
- added MX24: Right, MX_Alps_Hybrid:MX-1U-NoLED, F.Cu at (-536.4, 164.2)
- added MX25: F1, MX_Alps_Hybrid:MX-1U-NoLED, F.Cu at (-493.6, 69.0)
- added MX26: `, MX_Alps_Hybrid:MX-1U-NoLED, F.Cu at (-498.3, 88.0)
- added MX27: TAB, MX_Alps_Hybrid:MX-1.5U-NoLED, F.Cu at (-507.9, 107.1)
- added MX28: CAPS, MX_Alps_Hybrid:MX-1.75U-NoLED, F.Cu at (-515.0, 126.1)
- added MX29: LSHIFT, MX_Alps_Hybrid:MX-2.25U-NoLED, F.Cu at (-524.5, 145.2)
- added MX30: LCTRL, MX_Alps_Hybrid:MX-1.25U-NoLED, F.Cu at (-515.0, 164.2)
- added MX31: F2, MX_Alps_Hybrid:MX-1U-NoLED, F.Cu at (-474.5, 69.0)
- added MX32: 1, MX_Alps_Hybrid:MX-1U-NoLED, F.Cu at (-479.2, 88.0)
- added MX33: Q, MX_Alps_Hybrid:MX-1U-NoLED, F.Cu at (-484.0, 107.1)
- added MX34: A, MX_Alps_Hybrid:MX-1U-NoLED, F.Cu at (-488.8, 126.1)
- added MX35: Z, MX_Alps_Hybrid:MX-1U-NoLED, F.Cu at (-493.5, 145.2)
- added MX36: LGUI, MX_Alps_Hybrid:MX-1.25U-NoLED, F.Cu at (-491.2, 164.2)
- added MX37: F3, MX_Alps_Hybrid:MX-1U-NoLED, F.Cu at (-261.4, 195.9)
- added MX38: 2, MX_Alps_Hybrid:MX-1U-NoLED, F.Cu at (-123.4, 53.3)
- added MX39: W, MX_Alps_Hybrid:MX-1U-NoLED, F.Cu at (-104.4, 33.1)
- added MX40: S, MX_Alps_Hybrid:MX-1U-NoLED, F.Cu at (-167.5, 93.7)
- added MX41: X, MX_Alps_Hybrid:MX-1U-NoLED, F.Cu at (-211.5, 134.1)
- added MX42: LALT, MX_Alps_Hybrid:MX-1.25U-NoLED, F.Cu at (-380.2, 139.5)
- added MX43: F4, MX_Alps_Hybrid:MX-1U-NoLED, F.Cu at (-281.6, 175.7)
- added MX44: 3, MX_Alps_Hybrid:MX-1U-NoLED, F.Cu at (-236.4, 154.9)
- added MX45: E, MX_Alps_Hybrid:MX-1U-NoLED, F.Cu at (-197.2, 113.9)
- added MX46: D, MX_Alps_Hybrid:MX-1U-NoLED, F.Cu at (-261.4, 175.7)
- added MX47: C, MX_Alps_Hybrid:MX-1U-NoLED, F.Cu at (-281.6, 195.9)
- added MX48: SPACE, MX_Alps_Hybrid:MX-2U-NoLED, F.Cu at (-280.3, 33.1)
- added MX49: F5, MX_Alps_Hybrid:MX-1U-NoLED, F.Cu at (-143.6, 53.3)
- added MX5: P1, MX_Alps_Hybrid:MX-1U-NoLED, F.Cu at (-656.5, 145.3)
- added MX50: 4, MX_Alps_Hybrid:MX-1U-NoLED, F.Cu at (-124.6, 33.1)
- added MX51: R, MX_Alps_Hybrid:MX-1U-NoLED, F.Cu at (-187.7, 93.7)
- added MX52: F, MX_Alps_Hybrid:MX-1U-NoLED, F.Cu at (-231.7, 134.7)
- added MX53: V, MX_Alps_Hybrid:MX-1U-NoLED, F.Cu at (-173.4, 73.5)
- added MX54: MO(1), MX_Alps_Hybrid:MX-1U-NoLED, F.Cu at (-256.6, 154.9)
- added MX55: F6, MX_Alps_Hybrid:MX-1U-NoLED, F.Cu at (-130.7, 134.1)
- added MX56: 5, MX_Alps_Hybrid:MX-1U-NoLED, F.Cu at (-144.8, 33.1)
- added MX57: T, MX_Alps_Hybrid:MX-1U-NoLED, F.Cu at (-207.9, 93.7)
- added MX58: G, MX_Alps_Hybrid:MX-1U-NoLED, F.Cu at (-251.9, 134.7)
- added MX59: B, MX_Alps_Hybrid:MX-1U-NoLED, F.Cu at (-193.6, 73.5)
- added MX6: P0, MX_Alps_Hybrid:MX-1U-NoLED, F.Cu at (-656.5, 164.3)
- added MX6: P0, MX_Alps_Hybrid:MX-2U-NoLED, F.Cu at (-646.9, 164.3)
- added MX60: VOLD, MX_Alps_Hybrid:MX-1U-NoLED, F.Cu at (-276.8, 155.5)
- added MX61: F7, MX_Alps_Hybrid:MX-1U-NoLED, F.Cu at (-301.8, 175.7)
- added MX62: 6, MX_Alps_Hybrid:MX-1U-NoLED, F.Cu at (-237.6, 114.5)
- added MX63: Y, MX_Alps_Hybrid:MX-1U-NoLED, F.Cu at (-184.0, 53.3)
- added MX64: H, MX_Alps_Hybrid:MX-1U-NoLED, F.Cu at (-165.0, 33.1)
- added MX65: N, MX_Alps_Hybrid:MX-1U-NoLED, F.Cu at (-141.9, 182.6)
- added MX66: VOLU, MX_Alps_Hybrid:MX-1U-NoLED, F.Cu at (-224.4, 53.3)
- added MX67: F8, MX_Alps_Hybrid:MX-1U-NoLED, F.Cu at (-213.8, 73.5)
- added MX68: 7, MX_Alps_Hybrid:MX-1U-NoLED, F.Cu at (-163.8, 53.3)
- added MX69: U, MX_Alps_Hybrid:MX-1U-NoLED, F.Cu at (-322.0, 179.9)
- added MX7: P*, MX_Alps_Hybrid:MX-1U-NoLED, F.Cu at (-618.4, 88.1)
- added MX70: J, MX_Alps_Hybrid:MX-1U-NoLED, F.Cu at (-257.8, 114.5)
- added MX71: M, MX_Alps_Hybrid:MX-1U-NoLED, F.Cu at (-204.2, 53.3)
- added MX72: SPACE, MX_Alps_Hybrid:MX-2.75U-NoLED, F.Cu at (-365.9, 33.1)
- added MX73: F9, MX_Alps_Hybrid:MX-1U-NoLED, F.Cu at (-185.2, 33.1)
- added MX74: 8, MX_Alps_Hybrid:MX-1U-NoLED, F.Cu at (-248.3, 94.3)
- added MX75: I, MX_Alps_Hybrid:MX-1U-NoLED, F.Cu at (-292.3, 135.3)
- added MX76: K, MX_Alps_Hybrid:MX-1U-NoLED, F.Cu at (-317.2, 155.5)
- added MX77: ,, MX_Alps_Hybrid:MX-1U-NoLED, F.Cu at (-234.0, 73.5)
- added MX78: RALT, MX_Alps_Hybrid:MX-1.25U-NoLED, F.Cu at (-296.9, 74.1)
- added MX79: F10, MX_Alps_Hybrid:MX-1U-NoLED, F.Cu at (-342.2, 179.9)
- added MX8: P9, MX_Alps_Hybrid:MX-1U-NoLED, F.Cu at (-618.4, 107.2)
- added MX80: 9, MX_Alps_Hybrid:MX-1U-NoLED, F.Cu at (-278.0, 114.5)
- added MX81: O, MX_Alps_Hybrid:MX-1U-NoLED, F.Cu at (-337.4, 159.7)
- added MX82: L, MX_Alps_Hybrid:MX-1U-NoLED, F.Cu at (-241.2, 195.3)
- added MX83: ., MX_Alps_Hybrid:MX-1U-NoLED, F.Cu at (-221.0, 175.1)
- added MX84: RGUI, MX_Alps_Hybrid:MX-1.25U-NoLED, F.Cu at (-341.0, 115.1)
- added MX85: F11, MX_Alps_Hybrid:MX-1U-NoLED, F.Cu at (-153.2, 73.5)
- added MX86: 0, MX_Alps_Hybrid:MX-1U-NoLED, F.Cu at (-147.3, 93.7)
- added MX87: P, MX_Alps_Hybrid:MX-1U-NoLED, F.Cu at (-264.8, 53.9)
- added MX88: ;, MX_Alps_Hybrid:MX-1U-NoLED, F.Cu at (-362.4, 179.9)
- added MX89: /, MX_Alps_Hybrid:MX-1U-NoLED, F.Cu at (-254.2, 74.1)
- added MX9: P8, MX_Alps_Hybrid:MX-1U-NoLED, F.Cu at (-637.4, 107.2)
- added MX90: MENU, MX_Alps_Hybrid:MX-1.25U-NoLED, F.Cu at (-355.2, 139.5)
- added MX91: F12, MX_Alps_Hybrid:MX-1U-NoLED, F.Cu at (-274.4, 74.1)
- added MX92: -, MX_Alps_Hybrid:MX-1U-NoLED, F.Cu at (-205.4, 33.1)
- added MX93: [, MX_Alps_Hybrid:MX-1U-NoLED, F.Cu at (-268.5, 94.3)
- added MX94: ', MX_Alps_Hybrid:MX-1U-NoLED, F.Cu at (-312.5, 135.3)
- added MX95: RSHIFT, MX_Alps_Hybrid:MX-1.75U-NoLED, F.Cu at (-336.2, 74.7)
- added MX96: RCTRL, MX_Alps_Hybrid:MX-1.25U-NoLED, F.Cu at (-248.2, 33.1)
- added MX97: PSCR, MX_Alps_Hybrid:MX-1U-NoLED, F.Cu at (-608.6, 61.3)
- added MX98: =, MX_Alps_Hybrid:MX-1U-NoLED, F.Cu at (-244.6, 53.3)
- added MX99: ], MX_Alps_Hybrid:MX-1U-NoLED, F.Cu at (-332.7, 135.3)
- added U2: Elite-C, Keebio-Parts:Elite-C-castellated-29pin-holes, F.Cu at (-534.0, 77.3)
- MX1: value MX-NoLED -> P/
- MX2: value MX-NoLED -> NLCK
- MX3: value MX-NoLED -> P7
- MX4: value MX-NoLED -> P4
- moved MX3 790.0 mm to (-656.5, 107.2), turned to 0 degrees
- moved MX4 790.0 mm to (-656.5, 126.2)
- moved D4 788.7 mm to (-646.9, 126.2)
- moved D3 788.5 mm to (-646.9, 107.2)
- moved MX2 768.3 mm to (-656.5, 88.1)
- moved D2 767.1 mm to (-646.9, 88.1)
- moved MX1 750.4 mm to (-637.4, 88.1)
- moved D1 749.2 mm to (-627.9, 88.1)
Connections:
- D3 pad 1: Row0 -> Row2
- D4 pad 1: Row1 -> Row3
- MX1 pad 1: COl0 -> Col0
- MX2 pad 1: COl0 -> Col0
- MX3 pad 1: COl1 -> Col0
- MX4 pad 1: COl1 -> Col0
Routing:
- net GND: track 148.6 -> 0.00 mm, vias 22 -> 0
- net Row0: track 85.8 -> 0.00 mm, vias 4 -> 0
- net +5V: track 81.2 -> 0.00 mm, vias 11 -> 0
- net Row1: track 60.5 -> 0.00 mm, vias 3 -> 0
- net COl1: track 59.0 -> 0.00 mm, vias 3 -> 0
- net Net-(C3-Pad1): track 53.9 -> 0.00 mm, vias 7 -> 0
- net COl0: track 50.8 -> 0.00 mm, vias 2 -> 0
- net Net-(C4-Pad1): track 33.5 -> 0.00 mm, vias 2 -> 0
- net Net-(R2-Pad1): track 29.7 -> 0.00 mm, vias 2 -> 0
- net Net-(R1-Pad1): track 25.9 -> 0.00 mm, vias 2 -> 0
- net Net-(R3-Pad1): track 20.8 -> 0.00 mm, vias 4 -> 0
- net Net-(USB1-Pad6): track 16.3 -> 0.00 mm
- net Net-(D3-Pad2): track 14.4 -> 0.00 mm, vias 2 -> 0
- net Net-(C6-Pad1): track 11.4 -> 0.00 mm
- net Net-(D2-Pad2): track 9.78 -> 0.00 mm, vias 2 -> 0
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Other:
- board outline removed

Commit message: 1st angled col added
Parts:
- added MX28: CAPS, MX_Alps_Hybrid:MX-1.25U-NoLED, F.Cu at (-511.0, 126.2)
- moved D16 548.2 mm to (-608.8, 145.3), turned to 90 degrees
- moved D18 532.3 mm to (-589.8, 154.8), turned to 90 degrees
- moved D22 513.2 mm to (-566.0, 164.3), turned to 90 degrees
- moved D20 504.5 mm to (-566.0, 88.1), turned to 90 degrees
- moved D21 489.1 mm to (-546.9, 145.3), turned to 90 degrees
- moved D24 477.5 mm to (-527.8, 164.3), turned to 90 degrees
- moved D19 449.5 mm to (-513.5, 64.3), turned to 90 degrees
- moved D26 421.1 mm to (-489.7, 88.1), turned to 90 degrees
- moved MX97 420.3 mm to (-193.0, -1.65)
- moved D12 393.3 mm to (-627.9, 164.3), turned to 90 degrees
- moved MX39 362.5 mm to (-458.5, 110.6), turned to 345 degrees
- moved MX19 340.8 mm to (-523.0, 64.3)
- moved MX38 332.4 mm to (-453.5, 92.2), turned to 345 degrees
- moved D23 301.5 mm to (-546.9, 164.3), turned to 90 degrees
- moved MX40 298.1 mm to (-463.4, 129.0), turned to 345 degrees
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Connections:
- U2 pad 1: Net-(U2-Pad1) -> Col0
- U2 pad 10: Net-(U2-Pad10) -> Row0
- U2 pad 11: Net-(U2-Pad11) -> Row1
- U2 pad 12: Net-(U2-Pad12) -> Row2
- U2 pad 2: Net-(U2-Pad2) -> Col1
- U2 pad 25: Net-(U2-Pad25) -> Row3
- U2 pad 26: Net-(U2-Pad26) -> Row4
- U2 pad 27: Net-(U2-Pad27) -> Row5
- U2 pad 5: Net-(U2-Pad5) -> Col2
- U2 pad 6: Net-(U2-Pad6) -> Col3
- U2 pad 7: Net-(U2-Pad7) -> Col4
- U2 pad 8: Net-(U2-Pad8) -> Col5
- U2 pad 9: Net-(U2-Pad9) -> Col6
Routing:
- net Row2: track 0.00 -> 251.4 mm, vias 0 -> 12
- net Row1: track 0.00 -> 246.5 mm, vias 0 -> 12
- net Row3: track 0.00 -> 239.3 mm, vias 0 -> 13
- net Row0: track 0.00 -> 235.0 mm, vias 0 -> 13
- net Row5: track 0.00 -> 200.8 mm, vias 0 -> 4
- net Row4: track 0.00 -> 196.0 mm, vias 0 -> 8
- net Col3: track 0.00 -> 192.5 mm, vias 0 -> 3
- net Col4: track 0.00 -> 133.8 mm, vias 0 -> 4
- net Col2: track 0.00 -> 120.1 mm, vias 0 -> 2
- net Col5: track 0.00 -> 113.1 mm, vias 0 -> 2
- net Col0: track 0.00 -> 106.8 mm
- net Col1: track 0.00 -> 95.2 mm
- net Net-(D29-Pad2): track 0.00 -> 20.1 mm
- net Net-(D28-Pad2): track 0.00 -> 17.6 mm, vias 0 -> 2
- net Net-(D6-Pad2): track 0.00 -> 16.9 mm
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
Commit message: Aligned Left side and Flip Diodes
Deleted traces
Placed Diodes on back side of board
Parts:
- D1, D10, D100, D101, D102, D103, D104, D105, D106, D11, D12, D13, D14, D15, D16, D17, D18, D19, D2, D20, D21, D22, D23, D24, D25, D26, D27, D28, D29, D3, D30, D31, D32, D33, D34, D35, D36, D37, D38, D39, D4, D40, D41, D42, D43, D44, D45, D46, D47, D48, D49, D5, D50, D51, D52, D53, D54, D55, D56, D57, D58, D59, D6, D60, D61, D62, D63, D64, D65, D66, D67, D68, D69, D7, D70, D71, D72, D73, D74, D75, D76, D77, D78, D79, D8, D80, D81, D82, D83, D84, D85, D86, D87, D88, D89, D9, D90, D91, D92, D93, D94, D95, D96, D97, D98, D99: moved to B.Cu
- MX48: footprint MX_Alps_Hybrid:MX-2U-NoLED -> MX_Alps_Hybrid:MX-2.75U-NoLED
- moved D54 352.9 mm to (-383.7, 187.3), turned to 75 degrees
- moved MX50 297.9 mm to (-414.9, 100.0), turned to 345 degrees
- moved MX49 267.5 mm to (-410.2, 76.0), turned to 345 degrees
- moved MX53 264.8 mm to (-424.8, 156.5), turned to 345 degrees
- moved MX45 239.4 mm to (-436.6, 113.9), turned to 345 degrees
- moved MX51 231.9 mm to (-418.2, 118.8), turned to 345 degrees
- moved MX59 230.3 mm to (-406.4, 161.5), turned to 345 degrees
- moved MX44 205.7 mm to (-433.3, 95.1), turned to 345 degrees
- moved MX48 204.9 mm to (-427.5, 175.6), turned to 345 degrees
- moved MX52 189.7 mm to (-421.4, 137.8), turned to 345 degrees
- moved MX46 183.5 mm to (-439.8, 132.8), turned to 345 degrees
- moved MX43 180.4 mm to (-428.6, 71.1), turned to 345 degrees
- moved D37 170.2 mm to (-437.6, 67.8), turned to 75 degrees
- moved MX47 167.6 mm to (-443.2, 151.6), turned to 345 degrees
- moved D38 157.3 mm to (-442.3, 91.8), turned to 75 degrees
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Routing:
- net Row2: track 251.4 -> 0.00 mm, vias 12 -> 0
- net Row1: track 246.5 -> 0.00 mm, vias 12 -> 0
- net Row3: track 239.3 -> 0.00 mm, vias 13 -> 0
- net Row0: track 235.0 -> 0.00 mm, vias 13 -> 0
- net Row5: track 200.8 -> 0.00 mm, vias 4 -> 0
- net Row4: track 196.0 -> 0.00 mm, vias 8 -> 0
- net Col3: track 192.5 -> 0.00 mm, vias 3 -> 0
- net Col4: track 133.8 -> 0.00 mm, vias 4 -> 0
- net Col2: track 120.1 -> 0.00 mm, vias 2 -> 0
- net Col5: track 113.1 -> 0.00 mm, vias 2 -> 0
- net Col0: track 106.8 -> 0.00 mm
- net Col1: track 95.2 -> 0.00 mm
- net Net-(D29-Pad2): track 20.1 -> 0.00 mm
- net Net-(D28-Pad2): track 17.6 -> 0.00 mm, vias 2 -> 0
- net Net-(D6-Pad2): track 16.9 -> 0.00 mm
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
Commit message: Finished PCB
Parts:
- removed D100, D106: D_Small, Diode_SMD:D_SOD-123
- removed MX100: \, MX_Alps_Hybrid:MX-1U-NoLED
- removed MX106: ENTER, MX_Alps_Hybrid:MX-1U-NoLED
- MX105: footprint MX_Alps_Hybrid:MX-1U-NoLED -> MX_Alps_Hybrid:MX-1.5U-NoLED
- MX95: footprint MX_Alps_Hybrid:MX-1.75U-NoLED -> MX_Alps_Hybrid:MX-2.25U-NoLED
- moved MX55 353.8 mm to (-391.8, 81.4), turned to 345 degrees
- moved MX56 337.1 mm to (-396.5, 105.4), turned to 345 degrees
- moved MX65 286.6 mm to (-341.0, 162.0), turned to 15 degrees
- moved MX57 274.7 mm to (-399.8, 124.3), turned to 345 degrees
- moved MX64 274.1 mm to (-344.5, 143.2), turned to 15 degrees
- moved MX68 252.5 mm to (-333.0, 100.6), turned to 15 degrees
- moved MX63 250.0 mm to (-347.9, 124.4), turned to 15 degrees
- moved MX58 234.9 mm to (-403.0, 143.2), turned to 345 degrees
- moved MX66 233.1 mm to (-359.4, 166.9), turned to 15 degrees
- moved MX73 217.4 mm to (-319.6, 71.6), turned to 15 degrees
- moved D55 215.6 mm to (-382.6, 83.9), turned to 75 degrees
- moved MX71 214.1 mm to (-322.6, 157.0), turned to 15 degrees
- moved MX86 209.1 mm to (-270.4, 88.2)
- moved MX67 208.9 mm to (-338.0, 76.5), turned to 15 degrees
- moved MX85 206.6 mm to (-273.2, 64.3)
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Connections:
- U2 pad 13: Net-(U2-Pad13) -> Col9
- U2 pad 14: Net-(U2-Pad14) -> Col10
- U2 pad 15: Net-(U2-Pad15) -> Col11
- U2 pad 16: Net-(U2-Pad16) -> Col12
- U2 pad 17: Net-(U2-Pad17) -> Col13
- U2 pad 18: Net-(U2-Pad18) -> Col14
- U2 pad 19: Net-(U2-Pad19) -> Col15
- U2 pad 20: Net-(U2-Pad20) -> Col16
- U2 pad 24: Net-(U2-Pad24) -> Col17
- U2 pad 28: Net-(U2-Pad28) -> Col7
- U2 pad 29: Net-(U2-Pad29) -> Col8
Routing:
- net Row5: track 0.00 -> 641.0 mm, vias 0 -> 9
- net Row2: track 0.00 -> 575.1 mm, vias 0 -> 5
- net Row4: track 0.00 -> 567.3 mm, vias 0 -> 7
- net Row1: track 0.00 -> 533.6 mm, vias 0 -> 6
- net Row3: track 0.00 -> 521.5 mm, vias 0 -> 5
- net Row0: track 0.00 -> 495.2 mm, vias 0 -> 3
- net Col15: track 0.00 -> 452.6 mm, vias 0 -> 1
- net Col16: track 0.00 -> 442.5 mm, vias 0 -> 1
- net Col14: track 0.00 -> 405.8 mm
- net Col17: track 0.00 -> 392.2 mm
- net Col13: track 0.00 -> 386.1 mm
- net Col12: track 0.00 -> 347.2 mm, vias 0 -> 2
- net Col11: track 0.00 -> 340.9 mm, vias 0 -> 2
- net Col10: track 0.00 -> 324.7 mm, vias 0 -> 4
- net Col9: track 0.00 -> 294.1 mm, vias 0 -> 4
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Other:
- board outline added: 481.7 x 142.6 mm

Commit message: Microcontroller
Parts:
- removed U2: Elite-C, Keebio-Parts:Elite-C-castellated-29pin-holes
- added C1: 22pF, Capacitor_SMD:C_0805_2012Metric, F.Cu at (-556.3, 95.1)
- added C2: 22pF, Capacitor_SMD:C_0805_2012Metric, F.Cu at (-543.0, 95.2)
- added C3: 0.1uF, Capacitor_SMD:C_0805_2012Metric, F.Cu at (-529.7, 89.9)
- added C4: 0.1uF, Capacitor_SMD:C_0805_2012Metric, F.Cu at (-525.6, 89.9)
- added C5: 1uF, Capacitor_SMD:C_0805_2012Metric, F.Cu at (-536.0, 115.7)
- added C6: 0.1uF, Capacitor_SMD:C_0805_2012Metric, F.Cu at (-521.5, 89.9)
- added C7: 10uF, Capacitor_SMD:C_0805_2012Metric, F.Cu at (-517.5, 89.9)
- added F1: 500mA, Fuse:Fuse_1206_3216Metric, F.Cu at (-564.1, 63.6)
- added R1: 22, Resistor_SMD:R_0805_2012Metric, F.Cu at (-542.6, 74.2)
- added R2: 22, Resistor_SMD:R_0805_2012Metric, F.Cu at (-547.0, 74.2)
- added R3: 10k, Resistor_SMD:R_0805_2012Metric, F.Cu at (-565.5, 57.8)
- added R4: 10k, Resistor_SMD:R_0805_2012Metric, F.Cu at (-564.8, 116.2)
- added SW1: SW_Push, random-keyboard-parts:SKQG-1155865, F.Cu at (-556.7, 57.4)
- added U1: ATmega32U4-AU, Package_QFP:TQFP-44_10x10mm_P0.8mm, F.Cu at (-549.6, 115.2)
- added USB1: Molex-0548190589, random-keyboard-parts:Molex-0548190589, F.Cu at (-545.3, 58.5)
- added Y1: Crystal_GND24_Small, Crystal:Crystal_SMD_3225-4Pin_3.2x2.5mm, F.Cu at (-549.2, 95.1)
- moved D17 13.5 mm to (-608.8, 164.3), turned to 270 degrees
- moved D101 1.00 mm to (-228.5, 126.2)
- moved D102 1.00 mm to (-204.7, 145.3)
- moved D103 1.00 mm to (-204.7, 64.3)
- moved D104 1.00 mm to (-223.8, 88.1)
- moved D105 1.00 mm to (-214.2, 107.2)
- moved D84 1.00 mm to (-257.1, 164.4)
- moved D85 1.00 mm to (-283.7, 64.3)
- moved D86 1.00 mm to (-280.9, 88.2)
- moved D87 1.00 mm to (-271.4, 107.2)
- moved D88 1.00 mm to (-266.6, 126.2)
- moved D89 1.00 mm to (-266.6, 145.3)
- moved D90 1.00 mm to (-233.3, 164.4)
- moved D91 1.00 mm to (-264.6, 64.3)
- moved D92 1.00 mm to (-261.9, 88.2)
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Routing:
- net +5V: track 0.00 -> 396.0 mm, vias 0 -> 10
- net GND: track 0.00 -> 290.9 mm, vias 0 -> 12
- net Col13: track 386.1 -> 519.3 mm, vias 0 -> 6
- net Net-(R3-Pad2): track 0.00 -> 73.2 mm, vias 0 -> 2
- net Col14: track 405.8 -> 468.6 mm, vias 0 -> 6
- net Col15: track 452.6 -> 507.4 mm, vias 1 -> 6
- net Net-(R1-Pad1): track 0.00 -> 52.8 mm, vias 0 -> 2
- net Net-(R2-Pad1): track 0.00 -> 50.7 mm, vias 0 -> 2
- net Col8: track 273.2 -> 323.6 mm
- net Col17: track 392.2 -> 438.6 mm, vias 0 -> 1
- net Col2: track 168.3 -> 211.1 mm, vias 0 -> 1
- net Col4: track 204.9 -> 162.7 mm, vias 4 -> 1
- net Col12: track 347.2 -> 386.4 mm, vias 2 -> 3
- net Col11: track 340.9 -> 378.8 mm, vias 2 -> 3
- net Row0: track 495.2 -> 531.5 mm, vias 3 -> 7
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Other:
- board size 481.7 x 142.6 mm -> 480.4 x 142.2 mm

Commit message: Removed Tracks
Rework tracks
Parts:
- C1, C2, C3, C4, C5, C6, C7, F1, R1, R2, R3, R4, SW1, U1, USB1, Y1: moved to B.Cu
- moved R3 48.0 mm to (-564.1, 105.8), turned to 270 degrees
- moved R4 30.3 mm to (-534.6, 119.3)
- moved C5 27.6 mm to (-563.4, 118.9)
- moved C3 27.0 mm to (-556.4, 86.6), turned to 270 degrees
- moved C7 27.0 mm to (-544.3, 86.6), turned to 270 degrees
- moved C4 26.9 mm to (-552.3, 86.7), turned to 270 degrees
- moved C6 26.9 mm to (-548.3, 86.7), turned to 270 degrees
- moved R1 20.8 mm to (-563.3, 72.3), turned to 90 degrees
- moved USB1 15.4 mm to (-560.6, 56.6)
- moved C2 13.8 mm to (-556.4, 98.4)
- moved SW1 13.7 mm to (-546.1, 66.1), turned to 180 degrees
- moved C1 13.4 mm to (-543.2, 98.2)
- moved R2 11.9 mm to (-558.7, 72.2), turned to 90 degrees
- moved F1 9.02 mm to (-572.8, 66.2), turned to 90 degrees
- moved Y1 3.31 mm to (-550.2, 98.3), turned to 180 degrees
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Routing:
- net Row5: track 617.6 -> 0.00 mm, vias 11 -> 0
- net Row4: track 583.0 -> 0.00 mm, vias 9 -> 0
- net Row2: track 573.7 -> 0.00 mm, vias 7 -> 0
- net Row0: track 531.5 -> 0.00 mm, vias 7 -> 0
- net Col13: track 519.3 -> 0.00 mm, vias 6 -> 0
- net Row1: track 512.5 -> 0.00 mm, vias 5 -> 0
- net Col15: track 507.4 -> 0.00 mm, vias 6 -> 0
- net Row3: track 506.7 -> 0.00 mm, vias 8 -> 0
- net Col16: track 478.1 -> 0.00 mm, vias 3 -> 0
- net Col14: track 468.6 -> 0.00 mm, vias 6 -> 0
- net Col17: track 438.6 -> 0.00 mm, vias 1 -> 0
- net +5V: track 396.0 -> 0.00 mm, vias 10 -> 0
- net Col12: track 386.4 -> 0.00 mm, vias 3 -> 0
- net Col11: track 378.8 -> 0.00 mm, vias 3 -> 0
- net Col10: track 351.8 -> 0.00 mm, vias 2 -> 0
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
Commit message: Re-haul Schematics
Placed all SMD components on backside of PCB
Parts:
- removed the MX28 at (-515.9, 126.2)
- removed the MX6 at (-646.9, 164.3)
- added MX100: P0, MX_Alps_Hybrid:MX-2U-ReversedStabilizers-NoLED, F.Cu at (-646.9, 164.3)
- added MX106: CAPS, MX_Alps_Hybrid:MX-1.25U-NoLED, F.Cu at (-511.2, 126.2)
- MX28: footprint MX_Alps_Hybrid:MX-1.25U-NoLED -> MX_Alps_Hybrid:MX-1.75U-NoLED
- MX29: footprint MX_Alps_Hybrid:MX-2.25U-NoLED -> MX_Alps_Hybrid:MX-1U-NoLED
- MX48, MX72: footprint MX_Alps_Hybrid:MX-2.75U-NoLED -> MX_Alps_Hybrid:MX-2.75U-ReversedStabilizers-NoLED
- moved R4 31.9 mm to (-566.2, 114.3), turned to 0 degrees
- moved R3 30.4 mm to (-540.4, 86.7), turned to 90 degrees
- moved C5 29.3 mm to (-534.1, 117.2), turned to 90 degrees
- moved SW1 10.3 mm to (-540.6, 57.4)
- moved MX28 4.92 mm to (-516.0, 126.2)
- moved MX83 0.94 mm to (-285.9, 147.2)
- moved R1 0.53 mm to (-563.0, 71.8), turned to 0 degrees
- moved R2 0.51 mm to (-559.0, 71.8), turned to 180 degrees
- moved MX91 0.43 mm to (-254.7, 64.3)
- moved MX85 0.43 mm to (-273.7, 64.3)
- moved MX32 0.13 mm to (-480.3, 88.1)
- moved MX34 0.13 mm to (-489.8, 126.2)
- moved MX35 0.13 mm to (-494.5, 145.3)
- moved MX33 0.13 mm to (-485.0, 107.2)
- moved MX87 0.10 mm to (-261.8, 107.2)
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Connections:
- U1 pad 1: Col13 -> Col2
- U1 pad 10: Row2 -> Net-(U1-Pad10)
- U1 pad 36: Net-(U1-Pad36) -> Col13
- U1 pad 37: Col2 -> Col14
- U1 pad 41: Col14 -> Row2
Routing:
- net Row5: track 0.00 -> 602.3 mm, vias 0 -> 7
- net Row4: track 0.00 -> 543.0 mm, vias 0 -> 5
- net Row2: track 0.00 -> 529.5 mm, vias 0 -> 2
- net Row1: track 0.00 -> 527.6 mm
- net Col16: track 0.00 -> 525.7 mm, vias 0 -> 7
- net Col14: track 0.00 -> 510.4 mm, vias 0 -> 1
- net Row0: track 0.00 -> 496.3 mm, vias 0 -> 3
- net Row3: track 0.00 -> 484.0 mm, vias 0 -> 5
- net Col17: track 0.00 -> 472.9 mm, vias 0 -> 5
- net Col15: track 0.00 -> 464.0 mm, vias 0 -> 5
- net Col13: track 0.00 -> 439.0 mm, vias 0 -> 5
- net Col11: track 0.00 -> 357.1 mm, vias 0 -> 5
- net Col12: track 0.00 -> 345.9 mm, vias 0 -> 5
- net Col9: track 0.00 -> 322.4 mm, vias 0 -> 6
- net Col10: track 0.00 -> 312.9 mm
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Other:
- outline, holes or cut-outs redrawn
