File: HSC_Alice/HSC_Alice.kicad_pcb (KiCad board)
At the start: 2 copper layers, 480.4 x 142.2 mm, 226 parts, among them SW1 SW_Push, U1 ATmega32U4-AU, Y1 Crystal_GND24_Small

Commit message: Gerber Printed
Parts:
- F1: footprint Fuse:Fuse_1206_3216Metric -> Fuse:Fuse_0805_2012Metric
Changed lines of the file:
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@@
     (uvia_drill 0.1)
+  )
+  (module Fuse:Fuse_0805_2012Metric (layer B.Cu)
+    (at -572.77 66.1924 90)
+    (descr "Fuse SMD 0805 (2012 Metric), square (rectangular) end terminal, IPC_7351 nominal, (Body size source: https://docs.google.com/spreadsheets/d/1BsfQQcO9C6DZCsRaXUlFlo91Tg2WpOkGARC1WS5S8t0/edit?usp=sharing), generated with kicad-footprint-generator")
+    (tags fuse)
+    (attr smd)
+    (fp_text reference F1 (at 0 1.82 90) (layer B.SilkS)
+      (effects (font (size 1 1) (thickness 0.15)) (justify mirror))
+    )
+    (fp_text value 500mA (at 0 -1.82 90) (layer B.Fab)
+      (effects (font (size 1 1) (thickness 0.15)) (justify mirror))
+    )
+    (fp_text user %R (at 0 0 90) (layer B.Fab)
+      (effects (font (size 0.8 0.8) (thickness 0.12)) (justify mirror))
+    )
+    (fp_line (start -1 -0.6) (end -1 0.6) (layer B.Fab) (width 0.1))
+    (fp_line (start -1 0.6) (end 1 0.6) (layer B.Fab) (width 0.1))
+    (fp_line (start 1 0.6) (end 1 -0.6) (layer B.Fab) (width 0.1))
+    (fp_line (start 1 -0.6) (end -1 -0.6) (layer B.Fab) (width 0.1))
+    (fp_line (start -0.258578 0.71) (end 0.258578 0.71) (layer B.SilkS) (width 0.12))
+    (fp_line (start -0.258578 -0.71) (end 0.258578 -0.71) (layer B.SilkS) (width 0.12))
+    (fp_line (start -1.68 -0.95) (end -1.68 0.95) (layer B.CrtYd) (width 0.05))
+    (fp_line (start -1.68 0.95) (end 1.68 0.95) (layer B.CrtYd) (width 0.05))
+    (fp_line (start 1.68 0.95) (end 1.68 -0.95) (layer B.CrtYd) (width 0.05))
+    (fp_line (start 1.68 -0.95) (end -1.68 -0.95) (layer B.CrtYd) (width 0.05))
+    (pad 2 smd roundrect (at 0.9375 0 90) (size 0.975 1.4) (layers B.Cu B.Paste B.Mask) (roundrect_rratio 0.25)
+      (net 134 VCC))
+    (pad 1 smd roundrect (at -0.9375 0 90) (size 0.975 1.4) (layers B.Cu B.Paste B.Mask) (roundrect_rratio 0.25)
+      (net 132 +5V))
+    (model ${KISYS3DMOD}/Fuse.3dshapes/Fuse_0805_2012Metric.wrl
+      (at (xyz 0 0 0))
+      (scale (xyz 1 1 1))
+      (rotate (xyz 0 0 0))
+    )
   )
   (module MX_Alps_Hybrid:MX-1.5U-NoLED (layer F.Cu)
@@
       (effects (font (size 0.5 0.5) (thickness 0.08)) (justify mirror))
     )
-    (pad 2 smd roundrect (at 0.9125 0) (size 1.025 1.4) (layers B.Cu B.Paste B.Mask) (roundrect_rratio 0.2439014634146341)
+    (pad 2 smd roundrect (at 0.9125 0) (size 1.025 1.4) (layers B.Cu B.Paste B.Mask) (roundrect_rratio 0.2439004878048781)
       (net 140 "Net-(R4-Pad2)"))
-    (pad 1 smd roundrect (at -0.9125 0) (size 1.025 1.4) (layers B.Cu B.Paste B.Mask) (roundrect_rratio 0.2439014634146341)
+    (pad 1 smd roundrect (at -0.9125 0) (size 1.025 1.4) (layers B.Cu B.Paste B.Mask) (roundrect_rratio 0.2439004878048781)
       (net 129 GND))
     (model ${KISYS3DMOD}/Resistor_SMD.3dshapes/R_0805_2012Metric.wrl
@@
     (fp_line (start -1 0.625) (end 1 0.625) (layer B.Fab) (width 0.1))
     (fp_line (start -1 -0.625) (end -1 0.625) (layer B.Fab) (width 0.1))
-    (pad 1 smd roundrect (at -0.9125 0 90) (size 1.025 1.4) (layers B.Cu B.Paste B.Mask) (roundrect_rratio 0.2439014634146341)
+    (pad 1 smd roundrect (at -0.9125 0 90) (size 1.025 1.4) (layers B.Cu B.Paste B.Mask) (roundrect_rratio 0.2439004878048781)
       (net 132 +5V))
-    (pad 2 smd roundrect (at 0.9125 0 90) (size 1.025 1.4) (layers B.Cu B.Paste B.Mask) (roundrect_rratio 0.2439014634146341)
+    (pad 2 smd roundrect (at 0.9125 0 90) (size 1.025 1.4) (layers B.Cu B.Paste B.Mask) (roundrect_rratio 0.2439004878048781)
       (net 139 "Net-(R3-Pad2)"))
     (model ${KISYS3DMOD}/Resistor_SMD.3dshapes/R_0805_2012Metric.wrl
@@
       (effects (font (size 0.5 0.5) (thickness 0.08)) (justify mirror))
     )
-    (pad 2 smd roundrect (at 0.9125 0 180) (size 1.025 1.4) (layers B.Cu B.Paste B.Mask) (roundrect_rratio 0.2439014634146341)
+    (pad 2 smd roundrect (at 0.9125 0 180) (size 1.025 1.4) (layers B.Cu B.Paste B.Mask) (roundrect_rratio 0.2439004878048781)
       (net 137 D+))
-    (pad 1 smd roundrect (at -0.9125 0 180) (size 1.025 1.4) (layers B.Cu B.Paste B.Mask) (roundrect_rratio 0.2439014634146341)
+    (pad 1 smd roundrect (at -0.9125 0 180) (size 1.025 1.4) (layers B.Cu B.Paste B.Mask) (roundrect_rratio 0.2439004878048781)
       (net 138 "Net-(R2-Pad1)"))
     (model ${KISYS3DMOD}/Resistor_SMD.3dshapes/R_0805_2012Metric.wrl
@@
       (effects (font (size 0.5 0.5) (thickness 0.08)) (justify mirror))
     )
-    (pad 2 smd roundrect (at 0.9125 0) (size 1.025 1.4) (layers B.Cu B.Paste B.Mask) (roundrect_rratio 0.2439014634146341)
+    (pad 2 smd roundrect (at 0.9125 0) (size 1.025 1.4) (layers B.Cu B.Paste B.Mask) (roundrect_rratio 0.2439004878048781)
       (net 135 D-))
-    (pad 1 smd roundrect (at -0.9125 0) (size 1.025 1.4) (layers B.Cu B.Paste B.Mask) (roundrect_rratio 0.2439014634146341)
+    (pad 1 smd roundrect (at -0.9125 0) (size 1.025 1.4) (layers B.Cu B.Paste B.Mask) (roundrect_rratio 0.2439004878048781)
       (net 136 "Net-(R1-Pad1)"))
     (model ${KISYS3DMOD}/Resistor_SMD.3dshapes/R_0805_2012Metric.wrl
       (at (xyz 0 0 0))
       (scale (xyz 1 1 1))
-      (rotate (xyz 0 0 0))
-    )
-  )
-  (module Fuse:Fuse_1206_3216Metric (layer B.Cu)
-    (at -572.77 66.1924 90)
-    (descr "Fuse SMD 1206 (3216 Metric), square (rectangular) end terminal, IPC_7351 nominal, (Body size source: http://www.tortai-tech.com/upload/download/2011102023233369053.pdf), generated with kicad-footprint-generator")
-    (tags fuse)
-    (attr smd)
-    (fp_text reference F1 (at 0 1.82 90) (layer B.SilkS)
-      (effects (font (size 1 1) (thickness 0.15)) (justify mirror))
-    )
-    (fp_text value 500mA (at 0 -1.82 90) (layer B.Fab)
-      (effects (font (size 1 1) (thickness 0.15)) (justify mirror))
-    )
-    (fp_line (start -1.6 -0.8) (end -1.6 0.8) (layer B.Fab) (width 0.1))
-    (fp_line (start -1.6 0.8) (end 1.6 0.8) (layer B.Fab) (width 0.1))
-    (fp_line (start 1.6 0.8) (end 1.6 -0.8) (layer B.Fab) (width 0.1))
-    (fp_line (start 1.6 -0.8) (end -1.6 -0.8) (layer B.Fab) (width 0.1))
-    (fp_line (start -0.602064 0.91) (end 0.602064 0.91) (layer B.SilkS) (width 0.12))
-    (fp_line (start -0.602064 -0.91) (end 0.602064 -0.91) (layer B.SilkS) (width 0.12))
-    (fp_line (start -2.28 -1.12) (end -2.28 1.12) (layer B.CrtYd) (width 0.05))
-    (fp_line (start -2.28 1.12) (end 2.28 1.12) (layer B.CrtYd) (width 0.05))
-    (fp_line (start 2.28 1.12) (end 2.28 -1.12) (layer B.CrtYd) (width 0.05))
-    (fp_line (start 2.28 -1.12) (end -2.28 -1.12) (layer B.CrtYd) (width 0.05))
-    (fp_text user %R (at 0 0 90) (layer B.Fab)
-      (effects (font (size 0.8 0.8) (thickness 0.12)) (justify mirror))
-    )
-    (pad 2 smd roundrect (at 1.4 0 90) (size 1.25 1.75) (layers B.Cu B.Paste B.Mask) (roundrect_rratio 0.2)
-      (net 134 VCC))
-    (pad 1 smd roundrect (at -1.4 0 90) (size 1.25 1.75) (layers B.Cu B.Paste B.Mask) (roundrect_rratio 0.2)
-      (net 132 +5V))
-    (model ${KISYS3DMOD}/Fuse.3dshapes/Fuse_1206_3216Metric.wrl
-      (at (xyz 0 0 0))
-      (scale (xyz 1 1 1))
