File: HSC_Alice/HSC_Alice.kicad_pcb (KiCad board)
At the start: 2 copper layers, 479.3 x 144.1 mm, 211 parts, among them U2 Elite-C

Commit message: PCB Plate
Parts:
- MX48, MX72: footprint MX_Alps_Hybrid:MX-2.75U-NoLED -> MX_Alps_Hybrid:MX-2.75U-ReversedStabilizers-NoLED
Routing:
- net Net-(D72-Pad2): track 31.6 -> 34.3 mm
- net Net-(D48-Pad2): track 27.3 -> 25.9 mm
- net Col8: track 275.1 -> 276.3 mm
- net Col7: track 231.3 -> 230.1 mm
- net Col10: track 323.9 -> 325.1 mm

Commit message: Bug Fixes
Alignment, footprints and placement fixed
Parts:
- removed the MX28 at (-511.0, 126.2)
- removed the MX28 at (-515.9, 126.2)
- removed the MX6 at (-656.5, 164.3)
- added MX100: P0, MX_Alps_Hybrid:MX-1U-NoLED, F.Cu at (-656.4, 164.4)
- added MX106: CAPS, MX_Alps_Hybrid:MX-1.25U-FLIPPED, F.Cu at (-520.8, 126.2)
- added MX107: ENTER, MX_Alps_Hybrid:MX-ISO, F.Cu at (-198.6, 116.7)
- added MX28: CAPS, MX_Alps_Hybrid:MX-1.75U-NoLED, F.Cu at (-516.0, 126.2)
- MX48: footprint MX_Alps_Hybrid:MX-2.75U-ReversedStabilizers-NoLED -> MX_Alps_Hybrid:MX-2U-ReversedStabilizers-NoLED
- MX6: footprint MX_Alps_Hybrid:MX-2U-NoLED -> MX_Alps_Hybrid:MX-2U-ReversedStabilizers-NoLED
- U2: moved to B.Cu
- moved D6 9.52 mm to (-646.9, 154.8), turned to 180 degrees
- moved MX34 0.19 mm to (-489.8, 126.2)
- moved MX35 0.13 mm to (-494.5, 145.3)
- moved MX84 0.11 mm to (-246.3, 164.3)
- moved MX29 0.10 mm to (-525.5, 145.3)
- moved MX30 0.10 mm to (-516.0, 164.3)
- moved MX90 0.10 mm to (-222.4, 164.3)
- moved MX96 0.08 mm to (-198.6, 164.3)
- moved MX94 0.08 mm to (-239.1, 126.2)
- moved MX88 0.08 mm to (-258.2, 126.2)
- moved MX95 0.08 mm to (-227.2, 145.3)
- moved D102 0.06 mm to (-205.8, 145.3)
- moved D103 0.06 mm to (-205.8, 64.3)
- moved MX102 0.06 mm to (-196.2, 145.3)
- moved MX103 0.06 mm to (-196.2, 64.3)
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Connections:
- U2 pad 1: Col0 -> Col17
- U2 pad 10: Row0 -> Col4
- U2 pad 11: Row1 -> Col7
- U2 pad 12: Row2 -> Col8
- U2 pad 15: Col11 -> Col6
- U2 pad 16: Col12 -> Col5
- U2 pad 17: Col13 -> Row0
- U2 pad 18: Col14 -> Col3
- U2 pad 19: Col15 -> Col2
- U2 pad 2: Col1 -> Col16
- U2 pad 20: Col16 -> Col1
- U2 pad 24: Col17 -> Col0
- U2 pad 28: Col7 -> Row2
- U2 pad 29: Col8 -> Row1
- U2 pad 5: Col2 -> Col15
- U2 pad 6: Col3 -> Col14
- U2 pad 7: Col4 -> Col13
- U2 pad 8: Col5 -> Col12
- U2 pad 9: Col6 -> Col11
Routing:
- net Row5: track 637.4 -> 0.00 mm, vias 7 -> 0
- net Row2: track 575.9 -> 0.00 mm, vias 5 -> 0
- net Row4: track 557.8 -> 0.00 mm, vias 6 -> 0
- net Row1: track 529.6 -> 0.00 mm, vias 7 -> 0
- net Row3: track 519.0 -> 0.00 mm, vias 5 -> 0
- net Row0: track 496.9 -> 0.00 mm, vias 3 -> 0
- net Col15: track 452.4 -> 0.00 mm, vias 1 -> 0
- net Col16: track 438.9 -> 0.00 mm, vias 1 -> 0
- net Col14: track 404.6 -> 0.00 mm
- net Col17: track 392.0 -> 0.00 mm
- net Col13: track 385.9 -> 0.00 mm
- net Col12: track 349.0 -> 0.00 mm, vias 2 -> 0
- net Col11: track 342.7 -> 0.00 mm, vias 2 -> 0
- net Col10: track 325.1 -> 0.00 mm, vias 4 -> 0
- net Col9: track 292.4 -> 0.00 mm, vias 4 -> 0
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Other:
- board size 479.3 x 144.1 mm -> 479.2 x 142.2 mm

Commit message: Layout edit
Parts:
- MX106: footprint MX_Alps_Hybrid:MX-1.25U-FLIPPED -> MX_Alps_Hybrid:MX-1.25U-NoLED
- MX48: footprint MX_Alps_Hybrid:MX-2U-ReversedStabilizers-NoLED -> MX_Alps_Hybrid:MX-2.75U-ReversedStabilizers-NoLED
- moved MX38 7.85 mm to (-443.8, 90.7)
- moved MX39 6.24 mm to (-448.8, 109.1)
- moved MX37 3.16 mm to (-443.8, 66.9)
- moved MX40 2.98 mm to (-461.1, 128.0)
- moved MX72 2.94 mm to (-335.5, 180.5)
- moved MX78 2.94 mm to (-298.7, 170.7)
- moved D54 0.89 mm to (-383.1, 187.9)
- moved D60 0.89 mm to (-378.2, 169.5)
- moved MX42 0.69 mm to (-463.6, 166.3)
- moved D42 0.69 mm to (-452.1, 169.4)
- moved D48 0.66 mm to (-401.5, 183.0)
- moved MX48 0.66 mm to (-426.8, 176.2)
- moved D41 0.63 mm to (-451.8, 149.8)
- moved D47 0.63 mm to (-433.4, 154.7)
- moved D59 0.63 mm to (-396.6, 164.6)
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